File: hardware/BirdNest_pcb/BirdNest_pcb.kicad_pcb (KiCad board)
At the start: 2 copper layers, 94 x 78.2 mm, 33 parts, among them J1 Solarpanel, J2 AM312 connector, Q1 FQP27P06, Q5 FQP27P06, U1 DS18B20, U4 ESP32-CAM, U5 TP4056_Module, U6 VXO7803-500

Commit message: Update BirdNest firmware and PCB design
Parts:
- C2: footprint Capacitor_THT:CP_Radial_D8.0mm_P3.50mm -> Capacitor_THT:CP_Radial_D6.3mm_P2.50mm
- C3, C5: footprint Capacitor_THT:C_Disc_D5.0mm_W2.5mm_P5.00mm -> Capacitor_THT:C_Disc_D5.0mm_W2.5mm_P2.50mm
- moved C5 2.50 mm to (127.5, 105.0)
- moved C3 0.75 mm to (181.2, 83.5)
