File: hardware/BirdNest_pcb/BirdNest_pcb.kicad_sch (KiCad schematic)
At the start: 33 parts, among them J1 Solarpanel, J2 AM312 connector, Q1 FQP27P06, Q5 FQP27P06, U1 DS18B20, U4 ESP32-CAM, U5 TP4056_Module, U6 VXO7803-500

Commit message: Update BirdNest firmware and PCB design
Parts:
- C2: footprint Capacitor_THT:CP_Radial_D8.0mm_P3.50mm -> Capacitor_THT:CP_Radial_D6.3mm_P2.50mm
- C3, C5: footprint Capacitor_THT:C_Disc_D5.0mm_W2.5mm_P5.00mm -> Capacitor_THT:C_Disc_D5.0mm_W2.5mm_P2.50mm
Changed lines of the file:
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@@
 		)
 		(instances
-			(project "ESP32CAM_odu"
+			(project "BirdNest_pcb"
 				(path "/89abeaff-1b65-4d32-a0bb-ec0f19967e6e"
 					(reference "R6")
@@
 		)
 		(instances
-			(project "ESP32CAM_odu"
+			(project "BirdNest_pcb"
 				(path "/89abeaff-1b65-4d32-a0bb-ec0f19967e6e"
 					(reference "C6")
@@
 		)
 		(instances
-			(project "ESP32CAM_odu"
+			(project "BirdNest_pcb"
 				(path "/89abeaff-1b65-4d32-a0bb-ec0f19967e6e"
 					(reference "#PWR05")
@@
 		)
 		(instances
-			(project "ESP32CAM_odu"
+			(project "BirdNest_pcb"
 				(path "/89abeaff-1b65-4d32-a0bb-ec0f19967e6e"
 					(reference "JP2")
@@
 		)
 		(instances
-			(project "ESP32CAM_odu"
+			(project "BirdNest_pcb"
 				(path "/89abeaff-1b65-4d32-a0bb-ec0f19967e6e"
 					(reference "#PWR01")
@@
 		)
 		(instances
-			(project "ESP32CAM_odu"
+			(project "BirdNest_pcb"
 				(path "/89abeaff-1b65-4d32-a0bb-ec0f19967e6e"
 					(reference "U1")
@@
 		)
 		(instances
-			(project "ESP32CAM_odu"
+			(project "BirdNest_pcb"
 				(path "/89abeaff-1b65-4d32-a0bb-ec0f19967e6e"
 					(reference "#PWR03")
@@
 		)
 		(instances
-			(project "ESP32CAM_odu"
+			(project "BirdNest_pcb"
 				(path "/89abeaff-1b65-4d32-a0bb-ec0f19967e6e"
 					(reference "R3")
@@
 		)
 		(instances
-			(project "ESP32CAM_odu"
+			(project "BirdNest_pcb"
 				(path "/89abeaff-1b65-4d32-a0bb-ec0f19967e6e"
 					(reference "BT1")
@@
 		)
 		(instances
-			(project "ESP32CAM_odu"
+			(project "BirdNest_pcb"
 				(path "/89abeaff-1b65-4d32-a0bb-ec0f19967e6e"
 					(reference "U6")
@@
 		)
 		(instances
-			(project "ESP32CAM_odu"
+			(project "BirdNest_pcb"
 				(path "/89abeaff-1b65-4d32-a0bb-ec0f19967e6e"
 					(reference "H2")
@@
 		)
 		(instances
-			(project "ESP32CAM_odu"
+			(project "BirdNest_pcb"
 				(path "/89abeaff-1b65-4d32-a0bb-ec0f19967e6e"
 					(reference "R1")
@@
 		)
 		(instances
-			(project "ESP32CAM_odu"
+			(project "BirdNest_pcb"
 				(path "/89abeaff-1b65-4d32-a0bb-ec0f19967e6e"
 					(reference "Q1")
@@
 		)
 		(instances
-			(project "ESP32CAM_odu"
+			(project "BirdNest_pcb"
 				(path "/89abeaff-1b65-4d32-a0bb-ec0f19967e6e"
 					(reference "J2")
@@
 		)
 		(instances
-			(project "ESP32CAM_odu"
+			(project "BirdNest_pcb"
 				(path "/89abeaff-1b65-4d32-a0bb-ec0f19967e6e"
 					(reference "#PWR09")
@@
 		)
 		(instances
-			(project "ESP32CAM_odu"
+			(project "BirdNest_pcb"
 				(path "/89abeaff-1b65-4d32-a0bb-ec0f19967e6e"
 					(reference "#PWR013")
@@
 		)
 		(instances
-			(project "ESP32CAM_odu"
+			(project "BirdNest_pcb"
 				(path "/89abeaff-1b65-4d32-a0bb-ec0f19967e6e"
 					(reference "TP2")
@@
 		)
 		(instances
-			(project "ESP32CAM_odu"
+			(project "BirdNest_pcb"
 				(path "/89abeaff-1b65-4d32-a0bb-ec0f19967e6e"
 					(reference "#FLG04")
@@
 		)
 		(instances
-			(project "ESP32CAM_odu"
+			(project "BirdNest_pcb"
 				(path "/89abeaff-1b65-4d32-a0bb-ec0f19967e6e"
 					(reference "JP3")
@@
 		)
 		(instances
-			(project "ESP32CAM_odu"
+			(project "BirdNest_pcb"
 				(path "/89abeaff-1b65-4d32-a0bb-ec0f19967e6e"
 					(reference "JP1")
@@
 		)
 		(instances
-			(project "ESP32CAM_odu"
+			(project "BirdNest_pcb"
 				(path "/89abeaff-1b65-4d32-a0bb-ec0f19967e6e"
 					(reference "NT2")
@@
 		)
 		(instances
-			(project "ESP32CAM_odu"
+			(project "BirdNest_pcb"
 				(path "/89abeaff-1b65-4d32-a0bb-ec0f19967e6e"
 					(reference "#FLG05")
@@
 		)
 		(instances
-			(project "ESP32CAM_odu"
+			(project "BirdNest_pcb"
 				(path "/89abeaff-1b65-4d32-a0bb-ec0f19967e6e"
 					(reference "R10")
@@
 		)
 		(instances
-			(project "ESP32CAM_odu"
+			(project "BirdNest_pcb"
 				(path "/89abeaff-1b65-4d32-a0bb-ec0f19967e6e"
 					(reference "U4")
@@
 		)
 		(instances
-			(project "ESP32CAM_odu"
+			(project "BirdNest_pcb"
 				(path "/89abeaff-1b65-4d32-a0bb-ec0f19967e6e"
 					(reference "#PWR06")
@@
 		)
 		(instances
-			(project "ESP32CAM_odu"
+			(project "BirdNest_pcb"
 				(path "/89abeaff-1b65-4d32-a0bb-ec0f19967e6e"
 					(reference "J1")
@@
 		)
 		(instances
-			(project "ESP32CAM_odu"
+			(project "BirdNest_pcb"
 				(path "/89abeaff-1b65-4d32-a0bb-ec0f19967e6e"
 					(reference "#PWR08")
@@
 		)
 		(instances
-			(project "ESP32CAM_odu"
+			(project "BirdNest_pcb"
 				(path "/89abeaff-1b65-4d32-a0bb-ec0f19967e6e"
 					(reference "H1")
@@
 		)
 		(instances
-			(project "ESP32CAM_odu"
+			(project "BirdNest_pcb"
 				(path "/89abeaff-1b65-4d32-a0bb-ec0f19967e6e"
 					(reference "#FLG01")
@@
 		)
 		(instances
-			(project "ESP32CAM_odu"
+			(project "BirdNest_pcb"
 				(path "/89abeaff-1b65-4d32-a0bb-ec0f19967e6e"
 					(reference "R14")
@@
 		)
 		(instances
-			(project "ESP32CAM_odu"
+			(project "BirdNest_pcb"
 				(path "/89abeaff-1b65-4d32-a0bb-ec0f19967e6e"
 					(reference "#PWR018")
@@
 			)
 		)
-		(property "Footprint" "Capacitor_THT:CP_Radial_D8.0mm_P3.50mm"
+		(property "Footprint" "Capacitor_THT:CP_Radial_D6.3mm_P2.50mm"
 			(at 157.48 96.8248 0)
 			(hide yes)
@@
 		)
 		(instances
-			(project "ESP32CAM_odu"
+			(project "BirdNest_pcb"
 				(path "/89abeaff-1b65-4d32-a0bb-ec0f19967e6e"
 					(reference "C2")
@@
 		)
 		(instances
-			(project "ESP32CAM_odu"
+			(project "BirdNest_pcb"
 				(path "/89abeaff-1b65-4d32-a0bb-ec0f19967e6e"
 					(reference "H4")
@@
 		)
 		(instances
-			(project "ESP32CAM_odu"
+			(project "BirdNest_pcb"
 				(path "/89abeaff-1b65-4d32-a0bb-ec0f19967e6e"
 					(reference "#PWR07")
@@
 		)
 		(instances
-			(project "ESP32CAM_odu"
+			(project "BirdNest_pcb"
 				(path "/89abeaff-1b65-4d32-a0bb-ec0f19967e6e"
 					(reference "#PWR017")
@@
 		)
 		(instances
-			(project "ESP32CAM_odu"
+			(project "BirdNest_pcb"
 				(path "/89abeaff-1b65-4d32-a0bb-ec0f19967e6e"
 					(reference "Q5")
@@
 		)
 		(instances
-			(project "ESP32CAM_odu"
+			(project "BirdNest_pcb"
 				(path "/89abeaff-1b65-4d32-a0bb-ec0f19967e6e"
 					(reference "C1")
@@
 		)
 		(instances
-			(project "ESP32CAM_odu"
+			(project "BirdNest_pcb"
 				(path "/89abeaff-1b65-4d32-a0bb-ec0f19967e6e"
 					(reference "#PWR02")
@@
 		)
 		(instances
-			(project "ESP32CAM_odu"
+			(project "BirdNest_pcb"
 				(path "/89abeaff-1b65-4d32-a0bb-ec0f19967e6e"
 					(reference "D2")
@@
 		)
 		(instances
-			(project "ESP32CAM_odu"
+			(project "BirdNest_pcb"
 				(path "/89abeaff-1b65-4d32-a0bb-ec0f19967e6e"
 					(reference "TP1")
@@
 		)
 		(instances
-			(project "ESP32CAM_odu"
+			(project "BirdNest_pcb"
 				(path "/89abeaff-1b65-4d32-a0bb-ec0f19967e6e"
 					(reference "U5")
@@
 			)
 		)
-		(property "Footprint" "Capacitor_THT:C_Disc_D5.0mm_W2.5mm_P5.00mm"
+		(property "Footprint" "Capacitor_THT:C_Disc_D5.0mm_W2.5mm_P2.50mm"
 			(at 209.55 89.2048 0)
 			(hide yes)
@@
 		)
 		(instances
-			(project "ESP32CAM_odu"
+			(project "BirdNest_pcb"
 				(path "/89abeaff-1b65-4d32-a0bb-ec0f19967e6e"
 					(reference "C3")
@@
 		)
 		(instances
-			(project "ESP32CAM_odu"
+			(project "BirdNest_pcb"
 				(path "/89abeaff-1b65-4d32-a0bb-ec0f19967e6e"
 					(reference "R4")
@@
 		)
 		(instances
-			(project "ESP32CAM_odu"
+			(project "BirdNest_pcb"
 				(path "/89abeaff-1b65-4d32-a0bb-ec0f19967e6e"
 					(reference "R2")
@@
 		)
 		(instances
-			(project "ESP32CAM_odu"
+			(project "BirdNest_pcb"
 				(path "/89abeaff-1b65-4d32-a0bb-ec0f19967e6e"
 					(reference "#PWR04")
@@
 		)
 		(instances
-			(project "ESP32CAM_odu"
+			(project "BirdNest_pcb"
 				(path "/89abeaff-1b65-4d32-a0bb-ec0f19967e6e"
 					(reference "H3")
@@
 		)
 		(instances
-			(project "ESP32CAM_odu"
+			(project "BirdNest_pcb"
 				(path "/89abeaff-1b65-4d32-a0bb-ec0f19967e6e"
 					(reference "TP3")
@@
 			)
 		)
-		(property "Footprint" "Capacitor_THT:C_Disc_D5.0mm_W2.5mm_P5.00mm"
+		(property "Footprint" "Capacitor_THT:C_Disc_D5.0mm_W2.5mm_P2.50mm"
 			(at 174.9552 36.83 0)
 			(hide yes)
@@
 		)
 		(instances
-			(project "ESP32CAM_odu"
+			(project "BirdNest_pcb"
 				(path "/89abeaff-1b65-4d32-a0bb-ec0f19967e6e"
 					(reference "C5")
