File: hardware/BirdNest_pcb/BirdNest_pcb.kicad_sch (KiCad schematic)
At the start: 47 parts, among them J2 AM312 connector, J3 Solarpanel, Q6 FQP27P06, Q7 DMG2305UX, Q8 DMG2305UX, U1 DS18B20, U2 TP4056_Module, U3 ME2188, U4 ESP32-CAM, U7 LM393, U8 TL431DBZ

Commit message: Integrate release and local hardware updates into main
Co-authored-by: Copilot <223556219+Copilot@users.noreply.github.com>
Parts:
- removed J3: Solarpanel, TerminalBlock_Phoenix:TerminalBlock_Phoenix_MKDS-1,5-2-5.08_1x02_P5.08mm_Horizontal, symbol Connector:Conn_01x02_Pin
- removed U2: TP4056_Module, MyFootprints:TP4056-Module, symbol TP4056:TP4056
- added BT2, BT3: Battery, 1042:BAT_1042, symbol Batteryholder:1042
- added C13, C15, C18, C23, C24, C5: 10uF, symbol Device:C
- added C14, C16, C17, C19, C25, C4: 100nF, symbol Device:C
- added C22: 100nF, Capacitor_SMD:C_1206_3216Metric_Pad1.33x1.80mm_HandSolder, symbol Device:C
- added D10: SS34, Diode_SMD:D_SMA, symbol Diode:SS34
- added D4, D7: LED GREEN, symbol Device:LED
- added D5, D8: LED RED, symbol Device:LED
- added D9: SMAJ90CA, Diode_SMD:D_SMA, symbol Diode:SMAJ90CA
- added J4: Solarpanel, TerminalBlock_Phoenix:TerminalBlock_Phoenix_MKDS-1,5-2-5.08_1x02_P5.08mm_Horizontal, symbol Connector:Conn_01x02_Pin
- added Q2, Q3: FS8205A, FS8205A:SOP65P640X120-8N, symbol FS8205A:FS8205A
- added Q9: DMG2305UX, DMG2305UX:SOT23, symbol Transistor_FET:Q_PMOS_GSD
- added R10, R8: 1k, symbol Device:R
- added R11, R9: 100R, symbol Device:R
- added R12, R5: R, symbol Device:R
- added R13, R7: 330R, Resistor_SMD:R_1206_3216Metric_Pad1.30x1.75mm_HandSolder, symbol Device:R
- added R27: 100k, Resistor_SMD:R_1206_3216Metric_Pad1.30x1.75mm_HandSolder, symbol Device:R
- added R28, R30: 1M, Resistor_SMD:R_1206_3216Metric_Pad1.30x1.75mm_HandSolder, symbol Device:R
- added R29: 2M, Resistor_SMD:R_1206_3216Metric_Pad1.30x1.75mm_HandSolder, symbol Device:R
- added U10, U9: DW01A, Package_TO_SOT_SMD:SOT-23-6, symbol Battery_Management:DW01A
- added U11, U6: CN3065, CN3065:DFN300X300X90-9N, symbol CN3065:CN3065
Connections:
- net BAT_MON: now also C22.1, R29.2, R30.1
- net BAT_RAW: now also Q9.3 (D), R29.1
- net GND: now also BT2.N, C13.2, C14.2, C15.2, C16.2, C18.2, C22.2, C23.2, C24.2, C25.2, C4.2, C5.2, D9.1 (A1), J4.2 (Pin_2), Q2.2, Q2.3, R12.1, R30.2, R5.1, R8.2, U11.1 (TEMP), U11.3 (GND), U6.1 (TEMP), U6.3 (GND); no longer BT1.N
- net at Q7.2 (S), R20.2: now also BT2.P; no longer BT1.P
- new net: R5.2, U6.2 (ISET)
- new net: Q9.1 (G), R27.1, R28.1
- new net: R10.1, U10.2 (CS)
- new net: Q3.2, Q3.3, R10.2
- new net: D10.2 (A), D9.2 (A2), J4.1 (Pin_1)
- new net: D4.2 (A), D5.2 (A), R7.1
- new net: Q3.1, Q3.8
- new net: Q3.4, U10.3 (OC)
- new net: Q3.5, U10.1 (OD)
- new net: R8.1, U9.2 (CS)
- new net: Q2.1, Q2.8
- new net: Q2.4, U9.3 (OC)
- new net: Q2.5, U9.1 (OD)
- new net: C19.1, R11.1, U10.5 (VCC)
- new net: C17.1, R9.1, U9.5 (VCC)
- new net: D7.2 (A), D8.2 (A), R13.1
- new net: R12.2, U11.2 (ISET)
- new net B+: BT1.P, C13.1, C14.1, C18.1, R9.2, U6.5 (BAT), U6.8 (FB)
- new net B-: BT1.N, C17.2, Q2.6, Q2.7, U9.6 (GND)
- new net BAT+: BT3.P, C15.1, C16.1, C23.1, Q9.2 (S), R11.2, R28.2, U11.5 (BAT), U11.8 (FB)
- new net BAT-: BT3.N, C19.2, Q3.6, Q3.7, R27.2, U10.6 (GND)
- new net CHARGE: D5.1 (K), D8.1 (K), U11.7 (~{CHRG}), U6.7 (~{CHRG})
- new net C_DONE: D4.1 (K), D7.1 (K), U11.6 (~{DONE}), U6.6 (~{DONE})
- new net VCC: C24.1, C25.1, C4.1, C5.1, D10.1 (K), R13.2, R7.2, U11.4 (VIN), U6.4 (VIN)
- no-connect marks 14 -> 15
Other:
- moved on the sheet: C21, Q7, R20, R21, R24, R26
